File: Placa_DetectorParticulas/04_GenVref.kicad_sch (KiCad schematic)
At the start: 15 parts, among them U21 ADR5044WBRTZ-R7, U23 TSZ122IQ2T, U25 ADR5044WBRTZ-R7, U8 MCP4561T-104E/MF, U9 TSZ122IQ2T

Commit message: Dual Pot added.
Parts:
- removed C24: 100nF, Capacitor_SMD:C_0805_2012Metric, symbol Device:C
- removed U8: MCP4561T-104E/MF, DFN8_3x3MC_MCH, symbol 0A_MCP4561T_104E_MF:MCP4561T-104E_MF
- added C57: 100nF, Capacitor_SMD:C_0805_2012Metric, symbol Device:C
- added R79: 1k, Resistor_SMD:R_0805_2012Metric, symbol Device:R
- added R80, R81: 0, Resistor_SMD:R_0805_2012Metric, symbol Device:R
- added U29: MCP4661T-104E/ML, 0A_MCP4661T_104E_ML:QFN16_4x4MC_MCH, symbol 0A_MCP4661T_104E_ML:MCP4661T-104E_ML
- R16: value 5.1k -> 0
- R4: value 6.8k -> 4.7k
Connections:
- net +5V: now also C57.1, R81.1, U29.15 (VDD)
- net GND: now also C57.2, R80.1, U29.10 (P0B), U29.13 (A2), U29.14 (A1), U29.16 (HVC/A0), U29.17 (EP), U29.3 (VSS), U29.4 (VSS), U29.5 (P1B)
- net I2C5V_SCL: now also U29.1 (SCL)
- net I2C5V_SDA: now also U29.2 (SDA)
- net at R4.1, U21.1 (V+), U21.3 (NC): now also U29.7 (P1A), U29.8 (P0A)
- net at R32.1: now also U29.9 (P0W)
- net VREF1: now reaches U9.1 (OUT1), U9.2 (IN1-)
- net VREF1: no longer U9.5 (IN2+)
- net VREF renamed VREF2
- new net: R80.2, R81.2, U29.12 (*WP)
- new net: R79.1, U29.6 (P1W)
- new net: R79.2, U9.5 (IN2+)
Other:
- moved on the sheet: C25, R32, R4, U21, U9
